Commit message: New test Values

File: bad_robot_urdf/urdf/brobot_body.xacro (robot description, xacro)
@@ -10,5 +10,5 @@
     <xacro:property name="real_bodywidth" value="0.2" />
     <xacro:property name="real_bodyheight" value="0.11" />
-    <xacro:property name="body_mass" value="10.0" />
+    <xacro:property name="body_mass" value="2.0" />
     <xacro:property name="bodyclearance" value="0.01" />  <!--clearance from bottom of box to ground-->
      <!--Sonar offset, needed because otherwise the system detects the floor  -->

File: bad_robot_urdf/urdf/wheels.xacro (robot description, xacro)
@@ -32,6 +32,6 @@
   <!-- <xacro:property name="axle_eff_limit" value="5.12766"/>
   <xacro:property name="axle_vel_limit" value="244.8696"/> -->
-  <xacro:property name="axle_eff_limit" value="5.12766"/>
-  <xacro:property name="axle_vel_limit" value="244.8696"/>
+  <xacro:property name="axle_eff_limit" value="1.12766"/>
+  <xacro:property name="axle_vel_limit" value="10.8696"/>
   <!-- These constants are used to simulate a Traxxas 2056 servo operated at
        6 V. servo_stall_torque is measured in N m. servo_no_load_speed is

Commit message: Reseting the robot now

File: bad_robot_urdf/urdf/brobot_body.xacro (robot description, xacro)
@@ -20,5 +20,5 @@
     <!-- Position of wheels to body -->
     <xacro:property name="front_offset" value="0.08" />
-    <xacro:property name="wheel_radius" value="0.033" />
+    <xacro:property name="wheel_radius" value="${0.14605/2}" />
     <xacro:property name="front_wheelX" value="${-wheel_radius+real_bodylen/2}" />
     <xacro:property name="rear_wheelX" value="${-wheel_radius+real_bodylen/2}" />

File: bad_robot_urdf/urdf/wheels.xacro (robot description, xacro)
@@ -10,6 +10,6 @@
        is a "zero offset" wheel. hex_hub_depth = tire_width / 2 -
        axle_length. -->
-  <xacro:property name="hub_dia" value="0.09652"/>
-  <xacro:property name="tire_dia" value="0.14605"/>
+  <xacro:property name="hub_dia" value="${0.09652}"/>
+  <xacro:property name="tire_dia" value="${0.14605}"/>
   <xacro:property name="tire_width" value="0.0889"/>
   <xacro:property name="wheel_mass" value="0.29"/>
