Commit message: diff wheel robot

File: bad_robot_urdf/urdf/brobot.xacro (robot description, xacro)
@@ -2,8 +2,8 @@
 <robot
      xmlns:xacro="http://www.ros.org/wiki/xacro" name="brobot">
-  <xacro:include filename="$(find bad_robot_urdf)/urdf/brobot_body.xacro" />
-  <xacro:include filename="$(find bad_robot_urdf)/urdf/imu.xacro" />
-  <xacro:include filename="$(find bad_robot_urdf)/urdf/lidar.xacro" />
-  <xacro:include filename="$(find bad_robot_urdf)/urdf/kinect.xacro" />
-  <xacro:include filename="$(find bad_robot_urdf)/urdf/camera.xacro" />
+  <xacro:include filename="$(find bad_robot_urdf)/urdf/brobot_body_test.xacro" />
+  <!-- <xacro:include filename="$(find bad_robot_urdf)/urdf/imu.xacro" /> -->
+  <!-- <xacro:include filename="$(find bad_robot_urdf)/urdf/lidar.xacro" /> -->
+  <!-- <xacro:include filename="$(find bad_robot_urdf)/urdf/kinect.xacro" />
+  <xacro:include filename="$(find bad_robot_urdf)/urdf/camera.xacro" />   -->
 </robot>

File: bad_robot_urdf/urdf/camera.xacro (robot description, xacro)
@@ -21,5 +21,5 @@
       </visual>
       <inertial>
-          <mass value="0.1" />
+          <mass value="0.001" />
           <origin xyz="0 0 0" rpy="0 0 0"/>
           <inertia ixx="0.0001" ixy="0" ixz="0" iyy="0.0001" iyz="0" izz="0.0001" />

File: bad_robot_urdf/urdf/kinect.xacro (robot description, xacro)
@@ -21,5 +21,5 @@
       </visual>
       <inertial>
-          <mass value="0.1" />
+          <mass value="0.001" />
           <origin xyz="0 0 0" rpy="0 0 0"/>
           <inertia ixx="0.0001" ixy="0" ixz="0" iyy="0.0001" iyz="0" izz="0.0001" />

File: bad_robot_urdf/urdf/wheels.xacro (robot description, xacro)
@@ -10,7 +10,7 @@
        is a "zero offset" wheel. hex_hub_depth = tire_width / 2 -
        axle_length. -->
-  <xacro:property name="hub_dia" value="${0.09652}"/>
-  <xacro:property name="tire_dia" value="${0.14605}"/>
-  <xacro:property name="tire_width" value="0.0889"/>
+  <xacro:property name="hub_dia" value="${0.03652}"/>
+  <xacro:property name="tire_dia" value="${0.06605}"/>
+  <xacro:property name="tire_width" value="0.0189"/>
   <xacro:property name="wheel_mass" value="0.29"/>
   <!-- <xacro:property name="hub_dia" value="0.06"/>

Commit message: first version of car simulation

File: bad_robot_urdf/urdf/brobot.xacro (robot description, xacro)
@@ -2,8 +2,8 @@
 <robot
      xmlns:xacro="http://www.ros.org/wiki/xacro" name="brobot">
-  <xacro:include filename="$(find bad_robot_urdf)/urdf/brobot_body_test.xacro" />
-  <!-- <xacro:include filename="$(find bad_robot_urdf)/urdf/imu.xacro" /> -->
-  <!-- <xacro:include filename="$(find bad_robot_urdf)/urdf/lidar.xacro" /> -->
-  <!-- <xacro:include filename="$(find bad_robot_urdf)/urdf/kinect.xacro" />
-  <xacro:include filename="$(find bad_robot_urdf)/urdf/camera.xacro" />   -->
+  <xacro:include filename="$(find bad_robot_urdf)/urdf/brobot_body.xacro" />
+  <xacro:include filename="$(find bad_robot_urdf)/urdf/imu.xacro" />
+  <xacro:include filename="$(find bad_robot_urdf)/urdf/lidar.xacro" />
+  <xacro:include filename="$(find bad_robot_urdf)/urdf/kinect.xacro" />
+  <xacro:include filename="$(find bad_robot_urdf)/urdf/camera.xacro" />
 </robot>

File: bad_robot_urdf/urdf/brobot_body.xacro (robot description, xacro)
@@ -10,5 +10,5 @@
     <xacro:property name="real_bodywidth" value="0.2" />
     <xacro:property name="real_bodyheight" value="0.11" />
-    <xacro:property name="body_mass" value="2.0" />
+    <xacro:property name="body_mass" value="3.0" />
     <xacro:property name="bodyclearance" value="0.01" />  <!--clearance from bottom of box to ground-->
      <!--Sonar offset, needed because otherwise the system detects the floor  -->
@@ -117,4 +117,22 @@
                     lr_reflect="-1" fr_reflect="-1"
                     x="${rear_wheelX}" y="${wheelY}" z="${wheelZ}"/>
+<!-- Wheel Parameter -->
+<!-- With 0.2 there is no real difference -->
+<!-- <gazebo reference="left_front_wheel">
+  <mu1>0.2</mu1>
+  <mu2>0.2</mu2>
+</gazebo>
+<gazebo reference="right_front_wheel">
+  <mu1>0.2</mu1>
+  <mu2>0.2</mu2>
+</gazebo>
+<gazebo reference="left_rear_wheel">
+  <mu1>0.2</mu1>
+  <mu2>0.2</mu2>
+</gazebo>
+<gazebo reference="right_rear_wheel">
+  <mu1>0.2</mu1>
+  <mu2>0.2</mu2>
+</gazebo> -->
 <!-- ################################################################################################# -->
 <!-- Sonar -->

File: bad_robot_urdf/urdf/lidar.xacro (robot description, xacro)
@@ -31,5 +31,5 @@
       </ray>
       <plugin name="gazebo_ros_head_hokuyo_controller" filename="libgazebo_ros_laser.so">
-        <topicName>/scan</topicName>
+        <topicName>/sensor_msgs/LaserScan</topicName>
         <frameName>lidar_link</frameName>
       </plugin>

File: bad_robot_urdf/urdf/wheels.xacro (robot description, xacro)
@@ -14,30 +14,7 @@
   <xacro:property name="tire_width" value="0.0189"/>
   <xacro:property name="wheel_mass" value="0.29"/>
-  <!-- <xacro:property name="hub_dia" value="0.06"/>
-  <xacro:property name="tire_dia" value="0.066"/>
-  <xacro:property name="tire_width" value="0.027"/>
-  <xacro:property name="wheel_mass" value="0.29"/> -->
-  <!-- The specifications for a Titan(R) 550 motor could not be found, so the
-       stall torque of a Mabuchi Motor(R) RS-550VC-7525 motor was used instead.
-       num_spur_gear_teeth = 68
-       num_pinion_gear_teeth = 19
-       final_gear_ratio = (num_spur_gear_teeth / num_pinion_gear_teeth) *
-         5.22 = 18.68
-       stall_torque = 0.549 N m
-       axle_eff_limit = ((2 * stall_torque) * final_gear_ratio) / 4 =
-         5.12766 N m
-       max_speed = 40 mph (30+ mph) = 17.8816 m/s
-       axle_vel_limit = (2 * pi) * (max_speed / (pi * tire_dia)) =
-         244.8696 rad/s -->
-  <!-- <xacro:property name="axle_eff_limit" value="5.12766"/>
-  <xacro:property name="axle_vel_limit" value="244.8696"/> -->
   <xacro:property name="axle_eff_limit" value="1.12766"/>
   <xacro:property name="axle_vel_limit" value="10.8696"/>
-  <!-- These constants are used to simulate a Traxxas 2056 servo operated at
-       6 V. servo_stall_torque is measured in N m. servo_no_load_speed is
-       measured in rad/s. -->
-  <!-- <xacro:property name="servo_stall_torque" value="0.5649"/>
-  <xacro:property name="servo_no_load_speed" value="4.553"/> -->
-    <xacro:property name="servo_stall_torque" value="0.5649"/>
+  <xacro:property name="servo_stall_torque" value="0.5649"/>
   <xacro:property name="servo_no_load_speed" value="4.553"/>
 <!-- Materials -->
